Commit message: add extra fixed frame at hip

File: urdf/cheetah.urdf.xacro (robot description, xacro)
@@ -48,4 +48,29 @@
         <child link="trunk_interia"/>
     </joint>
+  <!-- <link name="stand">
+      <visual>
+          <origin rpy="0 0 0" xyz="0 0 0"/>
+          <geometry>
+            <box size="0.10 0.10 0.26"/>
+          </geometry>
+          <material name="white_gray"/>
+      </visual>
+      <collision>
+      <origin rpy="0 0 0" xyz="0 0 0"/>
+        <geometry>
+          <box size="0.10 0.10 0.26"/>
+        </geometry>
+      </collision>
+      <inertial>
+          <origin rpy="0 0 0" xyz="0 0 0"/>
+          <mass value="10000"/>
+          <inertia ixx="10000" ixy="10000" ixz="10000" iyy="10000"  iyz="10000" izz="10000"/>
+      </inertial>
+  </link>
+  <joint name="stand_to_trunk" type="fixed">
+      <origin rpy="0 0 0" xyz="0 0 -0.130465"/>
+      <parent link="trunk"/>
+      <child link="stand"/>
+  </joint> -->
     <xacro:leg name="RL" mirror="-1" mirror_dae="False" front_hind="1" front_hind_dae="True">
         <origin rpy="0 0 0" xyz="${leg_offset_x} ${-leg_offset_y} 0"/>

File: urdf/leg.urdf.xacro (robot description, xacro)
@@ -66,4 +66,12 @@
             </inertial>
         </link>
+        <link name="${name}_hip0">
+            <origin rpy="0 0 0" xyz="${hip_com_x*front_hind} ${hip_com_y*mirror} ${hip_com_z}"/>
+        </link>
+        <joint name="${name}_hip_joint0" type="fixed">
+            <xacro:insert_block name="origin"/>
+            <parent link="trunk"/>
+            <child link="${name}_hip0"/>
+        </joint>
     <!-- //////////////////////thigh//////////////////// -->
         <joint name="${name}_thigh_joint" type="revolute">
